File: Bachelor_Main_PCB/USB_HUB.kicad_sch (KiCad schematic)
At the start: 16 parts, among them J11 M20-9990245, U6 USB2514B-I/M2, Y3 SG-210STF 24Mhz

Commit message: Fix hierarchal sheet naming for USB hub
Connections:
- net USB_HUB_IN_M renamed USB_HUB_IN_N
- net USB_HUB_OUT_1_M renamed USB_HUB_OUT_1_N
- net USB_HUB_OUT_2_M renamed USB_HUB_OUT_2_N
Changed lines of the file:
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@@
 		)
 	)
-	(hierarchical_label "USB_HUB_OUT_2_M"
+	(hierarchical_label "USB_HUB_OUT_2_N"
 		(shape bidirectional)
 		(at 158.75 90.17 0)
@@
 		)
 	)
-	(hierarchical_label "USB_HUB_OUT_1_M"
+	(hierarchical_label "USB_HUB_OUT_1_N"
 		(shape bidirectional)
 		(at 158.75 77.47 0)
@@
 		)
 	)
-	(hierarchical_label "USB_HUB_IN_M"
+	(hierarchical_label "USB_HUB_IN_N"
 		(shape bidirectional)
 		(at 102.87 82.55 180)
