File: Bachelor_Main_PCB/SD-Card_interface.kicad_sch (KiCad schematic)
At the start: 1 part, among them J11 F32Q-1A7H1-11022

Commit message: Update page settings for all sheets. Add title, revision, date, etc.
Other:
- company: (none) -> Developed for the Norwegian Institute for Nature Research
- title: (none) -> Audiograb hardware
Changed lines of the file:
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@@
 	(generator_version "9.0")
 	(paper "A4")
+	(title_block
+		(title "Audiograb hardware")
+		(date "2025-05-27")
+		(rev "1.0")
+		(company "Developed for the Norwegian Institute for Nature Research")
+	)
 	(text "VDD"
 		(exclude_from_sim no)
@@
 				(size 1.27 1.27)
 			)
-			(hide yes)
 		)
 	)
@@
 				(size 2.54 2.54)
 			)
-			(hide yes)
 		)
 	)
@@
 				(size 1.27 1.27)
 			)
-			(hide yes)
 		)
 	)
@@
 				(size 1.27 1.27)
 			)
-			(hide yes)
 		)
 	)
@@
 				(size 1.27 1.27)
 			)
-			(hide yes)
 		)
 	)
@@
 				(size 1.27 1.27)
 			)
-			(hide yes)
 		)
 	)
@@
 				(size 1.27 1.27)
 			)
-			(hide yes)
 		)
 	)
@@
 				(size 1.27 1.27)
 			)
-			(hide yes)
 		)
 	)
@@
 				(size 1.27 1.27)
 			)
-			(hide yes)
 		)
 	)
@@
 				(size 1.27 1.27)
 			)
-			(hide yes)
 		)
 	)
